File: hardware/prototipo/placa_aquisicao_e_filtros/placa_aquisicao_e_filtros.sch (KiCad schematic (older format))
At the start: 20 parts, among them J1 Conn_01x04, J2 Conn_02x04_Odd_Even, J3 Conn_01x02, U1 Opamp_Quad_Generic, U2 AD620

Commit message: Acquisition PCB prototype in development.
Parts:
- removed J2: Conn_02x04_Odd_Even, Connector_PinHeader_2.54mm:PinHeader_2x04_P2.54mm_Vertical, symbol Connector_Generic:Conn_02x04_Odd_Even
- removed unit 2 of U1
- removed unit 3 of U1
- added J4: Conn_02x04_Counter_Clockwise, Connector_PinHeader_2.54mm:PinHeader_2x04_P2.54mm_Vertical, symbol Connector_Generic:Conn_02x04_Counter_Clockwise
- added R10: 0R, Resistor_THT:R_Axial_DIN0207_L6.3mm_D2.5mm_P10.16mm_Horizontal, symbol Device:R
- added unit 5 of U1
- added unit 1 of U1
Connections:
- wire segments 105 -> 104
Changed lines of the file:
@@
 $Comp
 L Device:Opamp_Quad_Generic U1
-U 1 1 5BAC02AC
+U 2 1 5BAC02AC
 P 3100 3350
 F 0 "U1" H 3100 2983 50  0000 C CNN
@@
 F 2 "Package_DIP:DIP-14_W7.62mm" H 3100 3350 50  0001 C CNN
 F 3 "~" H 3100 3350 50  0001 C CNN
-	1    3100 3350
+	2    3100 3350
 	-1   0    0    1
 $EndComp
@@
 Wire Wire Line
 	3050 2800 2600 2800
-Connection ~ 2600 2800
-Wire Wire Line
-	2600 2800 2600 3350
 $Comp
 L power:GNDA #PWR0101
@@
 Text GLabel 4900 2850 0    50   Input ~ 0
 right_electrode
-Text GLabel 2500 2800 0    50   Input ~ 0
+Text GLabel 2550 2800 0    50   Input ~ 0
 ref_electrode
 Wire Wire Line
-	2500 2800 2600 2800
-Wire Wire Line
 	4900 1900 4950 1900
 Wire Wire Line
@@
 Wire Wire Line
 	4950 2850 4900 2850
-$Comp
-L Device:Opamp_Quad_Generic U1
-U 2 1 5BACC30B
-P 6050 5400
-F 0 "U1" H 6050 5675 50  0000 C CNN
-F 1 "Opamp_Quad_Generic" H 6050 5676 50  0001 C CNN
-F 2 "Package_DIP:DIP-14_W7.62mm" H 6050 5400 50  0001 C CNN
-F 3 "~" H 6050 5400 50  0001 C CNN
-	2    6050 5400
-	1    0    0    -1
-$EndComp
 Wire Wire Line
 	8300 2350 8600 2350
@@
 Wire Wire Line
 	8700 5100 8650 5100
-$Comp
-L Device:Opamp_Quad_Generic U1
-U 3 1 5BB27F8B
-P 8900 2450
-F 0 "U1" H 8858 2450 50  0000 L CNN
-F 1 "Opamp_Quad_Generic" H 8858 2405 50  0001 L CNN
-F 2 "Package_DIP:DIP-14_W7.62mm" H 8900 2450 50  0001 C CNN
-F 3 "~" H 8900 2450 50  0001 C CNN
-	3    8900 2450
-	1    0    0    -1
-$EndComp
 Wire Wire Line
 	5950 5050 5950 5100
@@
 Wire Wire Line
 	5350 2050 5350 2000
-$Comp
-L Device:Opamp_Quad_Generic U1
-U 4 1 5BAD8CA9
-P 6050 5400
-F 0 "U1" H 6008 5400 50  0001 L CNN
-F 1 "Opamp_Quad_Generic" H 6008 5355 50  0001 L CNN
-F 2 "Package_DIP:DIP-14_W7.62mm" H 6050 5400 50  0001 C CNN
-F 3 "~" H 6050 5400 50  0001 C CNN
-	4    6050 5400
-	1    0    0    -1
-$EndComp
 $Comp
 L Device:R_POT RV1
@@
 F 3 "~" H 4350 2200 50  0001 C CNN
 	1    4350 2200
-	1    0    0    -1
+	-1   0    0    1
 $EndComp
 Wire Wire Line
@@
 Wire Wire Line
 	4350 2750 4800 2750
-Wire Wire Line
-	4350 2400 4350 2350
-Wire Wire Line
-	3750 2000 4350 2000
-Wire Wire Line
-	4350 2050 4350 2000
-Connection ~ 4350 2000
-Wire Wire Line
-	4500 2200 4550 2200
-Wire Wire Line
-	4350 2000 4800 2000
-Wire Wire Line
-	4550 2200 4550 2400
-Wire Wire Line
-	4550 2400 4350 2400
-Connection ~ 4350 2400
 $Comp
 L power:GNDA #PWR0107
 U 1 1 5BAF842C
-P 2650 5300
-F 0 "#PWR0107" H 2650 5050 50  0001 C CNN
-F 1 "GNDA" H 2655 5127 50  0000 C CNN
-F 2 "" H 2650 5300 50  0001 C CNN
-F 3 "" H 2650 5300 50  0001 C CNN
-	1    2650 5300
-	1    0    0    -1
-$EndComp
-$Comp
-L power:GNDA #PWR0108
-U 1 1 5BAF8496
-P 1650 5300
-F 0 "#PWR0108" H 1650 5050 50  0001 C CNN
-F 1 "GNDA" H 1655 5127 50  0000 C CNN
-F 2 "" H 1650 5300 50  0001 C CNN
-F 3 "" H 1650 5300 50  0001 C CNN
-	1    1650 5300
-	1    0    0    -1
-$EndComp
-Wire Wire Line
-	1650 5300 1650 5250
-Wire Wire Line
-	1650 5250 1850 5250
-Wire Wire Line
-	2650 5300 2650 5250
-Wire Wire Line
-	2650 5250 2450 5250
+P 2650 5200
+F 0 "#PWR0107" H 2650 4950 50  0001 C CNN
+F 1 "GNDA" H 2655 5027 50  0000 C CNN
+F 2 "" H 2650 5200 50  0001 C CNN
+F 3 "" H 2650 5200 50  0001 C CNN
+	1    2650 5200
+	1    0    0    -1
+$EndComp
 $Comp
 L power:+9V #PWR0109
 U 1 1 5BB06501
-P 1800 5000
-F 0 "#PWR0109" H 1800 4850 50  0001 C CNN
-F 1 "+9V" H 1815 5173 50  0000 C CNN
-F 2 "" H 1800 5000 50  0001 C CNN
-F 3 "" H 1800 5000 50  0001 C CNN
-	1    1800 5000
-	1    0    0    -1
-$EndComp
-$Comp
-L power:+9V #PWR0110
-U 1 1 5BB0656B
-P 2500 5000
-F 0 "#PWR0110" H 2500 4850 50  0001 C CNN
-F 1 "+9V" H 2515 5173 50  0000 C CNN
-F 2 "" H 2500 5000 50  0001 C CNN
-F 3 "" H 2500 5000 50  0001 C CNN
-	1    2500 5000
-	1    0    0    -1
-$EndComp
-Wire Wire Line
-	2500 5000 2500 5050
-Wire Wire Line
-	2500 5050 2400 5050
-Wire Wire Line
-	1900 5050 1800 5050
-Wire Wire Line
-	1800 5050 1800 5000
-$Comp
-L power:-9V #PWR0111
-U 1 1 5BB0E1EE
+P 1850 5000
+F 0 "#PWR0109" H 1850 4850 50  0001 C CNN
+F 1 "+9V" H 1865 5173 50  0000 C CNN
+F 2 "" H 1850 5000 50  0001 C CNN
+F 3 "" H 1850 5000 50  0001 C CNN
+	1    1850 5000
+	1    0    0    -1
+$EndComp
+$Comp
+L power:-9V #PWR0112
+U 1 1 5BB0E288
 P 2450 5400
-F 0 "#PWR0111" H 2450 5275 50  0001 C CNN
+F 0 "#PWR0112" H 2450 5275 50  0001 C CNN
 F 1 "-9V" H 2465 5573 50  0000 C CNN
 F 2 "" H 2450 5400 50  0001 C CNN
@@
 	-1   0    0    1
 $EndComp
-$Comp
-L power:-9V #PWR0112
-U 1 1 5BB0E288
-P 1850 5400
-F 0 "#PWR0112" H 1850 5275 50  0001 C CNN
-F 1 "-9V" H 1865 5573 50  0000 C CNN
-F 2 "" H 1850 5400 50  0001 C CNN
-F 3 "" H 1850 5400 50  0001 C CNN
-	1    1850 5400
-	-1   0    0    1
-$EndComp
-Wire Wire Line
-	1850 5400 1850 5350
-Wire Wire Line
-	1850 5350 1900 5350
-Wire Wire Line
-	2400 5350 2450 5350
-Wire Wire Line
-	2450 5350 2450 5400
 $Comp
 L power:-9V #PWR0113
@@
 Wire Wire Line
 	2200 2250 2200 2300
-Wire Wire Line
-	1900 5150 1850 5150
-Wire Wire Line
-	1850 5150 1850 5250
-Connection ~ 1850 5250
-Wire Wire Line
-	1850 5250 1900 5250
-Wire Wire Line
-	2400 5150 2450 5150
-Wire Wire Line
-	2450 5150 2450 5250
-Connection ~ 2450 5250
-Wire Wire Line
-	2450 5250 2400 5250
-$Comp
-L Connector_Generic:Conn_02x04_Odd_Even J2
-U 1 1 5BB36384
+$Comp
+L Device:Opamp_Quad_Generic U1
+U 5 1 5BAD9E0E
+P 6050 5400
+F 0 "U1" H 6008 5400 50  0001 L CNN
+F 1 "Opamp_Quad_Generic" H 6008 5355 50  0001 L CNN
+F 2 "Package_DIP:DIP-14_W7.62mm" H 6050 5400 50  0001 C CNN
+F 3 "~" H 6050 5400 50  0001 C CNN
+	5    6050 5400
+	1    0    0    -1
+$EndComp
+$Comp
+L Device:Opamp_Quad_Generic U1
+U 1 1 5BAF0215
+P 8900 2450
+F 0 "U1" H 8900 2817 50  0000 C CNN
+F 1 "Opamp_Quad_Generic" H 8900 2726 50  0000 C CNN
+F 2 "Package_DIP:DIP-14_W7.62mm" H 8900 2450 50  0001 C CNN
+F 3 "~" H 8900 2450 50  0001 C CNN
+	1    8900 2450
+	1    0    0    -1
+$EndComp
+$Comp
+L Device:Opamp_Quad_Generic U1
+U 4 1 5BAF02E7
+P 6050 5400
+F 0 "U1" H 6050 5767 50  0000 C CNN
+F 1 "Opamp_Quad_Generic" H 6050 5676 50  0000 C CNN
+F 2 "Package_DIP:DIP-14_W7.62mm" H 6050 5400 50  0001 C CNN
+F 3 "~" H 6050 5400 50  0001 C CNN
+	4    6050 5400
+	1    0    0    -1
+$EndComp
+$Comp
+L Connector_Generic:Conn_02x04_Counter_Clockwise J4
+U 1 1 5BAF159D
 P 2100 5150
-F 0 "J2" H 2150 5467 50  0000 C CNN
-F 1 "Conn_02x04_Odd_Even" H 2150 5376 50  0000 C CNN
+F 0 "J4" H 2150 5375 50  0000 C CNN
+F 1 "Conn_02x04_Counter_Clockwise" H 2150 5376 50  0001 C CNN
 F 2 "Connector_PinHeader_2.54mm:PinHeader_2x04_P2.54mm_Vertical" H 2100 5150 50  0001 C CNN
 F 3 "~" H 2100 5150 50  0001 C CNN
@@
 	1    0    0    -1
 $EndComp
+Wire Wire Line
+	2450 5400 2450 5350
+Wire Wire Line
+	2450 5250 2400 5250
+Wire Wire Line
+	2400 5350 2450 5350
+Connection ~ 2450 5350
+Wire Wire Line
+	2450 5350 2450 5250
+Wire Wire Line
+	1850 5250 1900 5250
+Wire Wire Line
+	1900 5350 1850 5350
+Wire Wire Line
+	1850 5350 1850 5250
+Wire Wire Line
+	1850 5150 1900 5150
+Wire Wire Line
+	1900 5050 1850 5050
+Wire Wire Line
+	1850 5050 1850 5150
+Wire Wire Line
+	2650 5200 2650 5150
+Wire Wire Line
+	2400 5150 2450 5150
+Wire Wire Line
+	2400 5050 2450 5050
+Wire Wire Line
+	2450 5050 2450 5150
+Connection ~ 2450 5150
+Wire Wire Line
+	2450 5150 2650 5150
+Wire Wire Line
+	1850 5000 1850 5050
+Connection ~ 1850 5050
+$Comp
+L power:GNDA #PWR0108
+U 1 1 5BB2ADBE
+P 1850 5400
+F 0 "#PWR0108" H 1850 5150 50  0001 C CNN
+F 1 "GNDA" H 1855 5227 50  0000 C CNN
+F 2 "" H 1850 5400 50  0001 C CNN
+F 3 "" H 1850 5400 50  0001 C CNN
+	1    1850 5400
+	1    0    0    -1
+$EndComp
+Wire Wire Line
+	1850 5400 1850 5350
+Connection ~ 1850 5350
+$Comp
+L Device:R R10
+U 1 1 5BB2E561
+P 2600 3100
+F 0 "R10" H 2670 3146 50  0000 L CNN
+F 1 "0R" H 2670 3055 50  0000 L CNN
+F 2 "Resistor_THT:R_Axial_DIN0207_L6.3mm_D2.5mm_P10.16mm_Horizontal" V 2530 3100 50  0001 C CNN
+F 3 "~" H 2600 3100 50  0001 C CNN
+	1    2600 3100
+	1    0    0    -1
+$EndComp
+Wire Wire Line
+	2550 2800 2600 2800
+Connection ~ 2600 2800
+Wire Wire Line
+	2600 2950 2600 2800
+Wire Wire Line
+	2600 3350 2600 3250
+Wire Wire Line
+	3750 2000 4200 2000
+Wire Wire Line
+	4350 2400 4350 2350
+Wire Wire Line
+	4350 2050 4350 2000
+Connection ~ 4350 2000
+Wire Wire Line
+	4350 2000 4800 2000
+Wire Wire Line
+	4200 2200 4200 2000
+Connection ~ 4200 2000
+Wire Wire Line
+	4200 2000 4350 2000
 $EndSCHEMATC

Commit message: Acquisition prototype board finalized.
Parts:
- removed R10: 0R, Resistor_THT:R_Axial_DIN0207_L6.3mm_D2.5mm_P10.16mm_Horizontal, symbol Device:R
- added C6: 47u, Capacitors_THT:C_Disc_D6.0mm_W2.5mm_P5.00mm, symbol Device:C
- added R11: 130k, Resistors_THT:R_Axial_DIN0207_L6.3mm_D2.5mm_P10.16mm_Horizontal, symbol Device:R
- added R12: 18k, Resistors_THT:R_Axial_DIN0207_L6.3mm_D2.5mm_P10.16mm_Horizontal, symbol Device:R
- C1, C2, C3, C4, C5: symbol Device:C -> placa_aquisicao_e_filtros-rescue:C-Device
- J1: symbol Connector_Generic:Conn_01x04 -> placa_aquisicao_e_filtros-rescue:Conn_01x04-Connector_Generic
- J3: symbol Connector_Generic:Conn_01x02 -> placa_aquisicao_e_filtros-rescue:Conn_01x02-Connector_Generic
- J4: symbol Connector_Generic:Conn_02x04_Counter_Clockwise -> placa_aquisicao_e_filtros-rescue:Conn_02x04_Counter_Clockwise-Connector_Generic
- R1, R2, R3, R4, R5, R6, R7: symbol Device:R -> placa_aquisicao_e_filtros-rescue:R-Device
- R8: value 91k -> 33k; symbol Device:R -> placa_aquisicao_e_filtros-rescue:R-Device
- R9: value 47k -> 150k; symbol Device:R -> placa_aquisicao_e_filtros-rescue:R-Device
- RV1: symbol Device:R_POT -> placa_aquisicao_e_filtros-rescue:R_POT-Device
- U1: symbol Device:Opamp_Quad_Generic -> placa_aquisicao_e_filtros-rescue:Opamp_Quad_Generic-Device
- U2: symbol Amplifier_Instrumentation:AD620 -> placa_aquisicao_e_filtros-rescue:AD620-Amplifier_Instrumentation
Connections:
- wire segments 104 -> 109

Commit message: PCB with AGC routed but negative supply without voltage regulator
Parts:
- removed C4, C5: 47u, Capacitor_THT:C_Disc_D6.0mm_W2.5mm_P5.00mm, symbol placa_aquisicao_e_filtros-rescue:C-Device
- removed C6: 47u, Capacitors_THT:C_Disc_D6.0mm_W2.5mm_P5.00mm, symbol Device:C
- removed RV1: 1k, Potentiometer_THT:Potentiometer_Piher_PC-16_Single_Horizontal, symbol placa_aquisicao_e_filtros-rescue:R_POT-Device
- removed U1: Opamp_Quad_Generic, Package_DIP:DIP-14_W7.62mm, symbol placa_aquisicao_e_filtros-rescue:Opamp_Quad_Generic-Device
- added C1, C3, C6: 1u, Capacitor_THT:CP_Radial_D5.0mm_P2.50mm, symbol Device:CP
- added C10, C11: 47u, Capacitor_THT:CP_Radial_D5.0mm_P2.50mm, symbol Device:CP
- added C2, C5: 10u, Capacitor_THT:CP_Radial_D5.0mm_P2.50mm, symbol Device:CP
- added C9: 22u, Capacitor_THT:CP_Radial_D5.0mm_P2.50mm, symbol Device:CP
- added D1: 1N4148, Diode_THT:D_DO-35_SOD27_P7.62mm_Horizontal, symbol Diode:1N4148
- added J1: Conn_01x02, TerminalBlock:TerminalBlock_Altech_AK300-2_P5.00mm, symbol Connector_Generic:Conn_01x02
- added J4, J6: Conn_01x02, Connector_PinHeader_2.54mm:PinHeader_1x02_P2.54mm_Vertical, symbol Connector_Generic:Conn_01x02
- added Q1: BF245B, Package_TO_SOT_THT:TO-92_Inline_Wide, symbol Transistor_FET:BF245B
- added R10: 100k, Resistor_SMD:R_0805_2012Metric, symbol Device:R
- added R13: 22k, Resistor_SMD:R_0805_2012Metric, symbol Device:R
- added R14, R15: 1k, Resistor_SMD:R_0805_2012Metric, symbol Device:R
- added R17, R18, R8: 12k, Resistor_SMD:R_0805_2012Metric, symbol Device:R
- added R20: 68k, Resistor_SMD:R_0805_2012Metric, symbol Device:R
- added R21: 150k, Resistor_SMD:R_0805_2012Metric, symbol Device:R
- added R7: 560R, Resistor_SMD:R_0805_2012Metric, symbol Device:R
- added RV1: 470k, Potentiometer_THT:Potentiometer_ACP_CA6-H2,5_Horizontal, symbol Device:R_POT_TRIM
- added RV2: R_POT, Potentiometer_THT:Potentiometer_ACP_CA6-H2,5_Horizontal, symbol Device:R_POT
- added U1: AP1117-33, Package_TO_SOT_SMD:SOT-223-3_TabPin2, symbol Regulator_Linear:AP1117-33
- added U2: TPS60401, Package_TO_SOT_SMD:SOT-23-5, symbol tps60401:TPS60401
- added U3, U5: Opamp_Quad_Generic, Package_DIP:DIP-14_W7.62mm_Socket, symbol Device:Opamp_Quad_Generic
- C4: renamed from C2; footprint Capacitor_THT:C_Disc_D6.0mm_W2.5mm_P5.00mm -> Capacitor_THT:C_Rect_L7.2mm_W3.5mm_P5.00mm_FKS2_FKP2_MKS2_MKP2
- C8: renamed from C1; footprint Capacitor_THT:C_Disc_D6.0mm_W2.5mm_P5.00mm -> Capacitor_THT:C_Disc_D3.8mm_W2.6mm_P2.50mm
- R11: value 130k -> 200k; footprint Resistors_THT:R_Axial_DIN0207_L6.3mm_D2.5mm_P10.16mm_Horizontal -> Resistor_THT:R_Axial_DIN0207_L6.3mm_D2.5mm_P10.16mm_Horizontal
- R12: value 18k -> 51k; footprint Resistors_THT:R_Axial_DIN0207_L6.3mm_D2.5mm_P10.16mm_Horizontal -> Resistor_THT:R_Axial_DIN0207_L6.3mm_D2.5mm_P10.16mm_Horizontal
- R16: renamed from R8; value 33k -> 47k; footprint Resistor_THT:R_Axial_DIN0207_L6.3mm_D2.5mm_P10.16mm_Horizontal -> Resistor_SMD:R_0805_2012Metric
- R19: renamed from R9; value 150k -> 100k; footprint Resistor_THT:R_Axial_DIN0207_L6.3mm_D2.5mm_P10.16mm_Horizontal -> Resistor_SMD:R_0805_2012Metric
- R3: renamed from R1; footprint Resistor_THT:R_Axial_DIN0207_L6.3mm_D2.5mm_P10.16mm_Horizontal -> Resistor_SMD:R_0805_2012Metric
- R4: renamed from R2; value 10k -> 12k; footprint Resistor_THT:R_Axial_DIN0207_L6.3mm_D2.5mm_P10.16mm_Horizontal -> Resistor_SMD:R_0805_2012Metric
- R5: renamed from R3; value 24.9k -> 24k
- R6: renamed from R4; value 24.9k -> 24k
- R9: renamed from R5; footprint Resistor_THT:R_Axial_DIN0207_L6.3mm_D2.5mm_P10.16mm_Horizontal -> Resistor_SMD:R_0805_2012Metric
- U4: renamed from U2; footprint Package_DIP:DIP-8_W7.62mm -> Package_DIP:DIP-8_W7.62mm_Socket
- renumbered C3 to C7, J1 to J2, J4 to J3, J3 to J5, R6 to R1, R7 to R2
Connections:
- net labels added: +3V3, +Vin, -3V3, AGC, GNDA-power, HP, LP, OUT, SUM
- net labels removed: +9V, -9V, out1, out2, out3
- wire segments 109 -> 198
- no-connect marks 0 -> 1
Other:
- note added: "Automatic Gain Control"
- note added: "Somador de tensão"
- moved on the sheet: C4, C7, C8, J2, J3, J5, R1, R16, R19, R2, R3, R4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

Commit message: Second prototype working with bluetooth.
Parts:
- R14, R15: value 1k -> 1M
Connections:
- no-connect marks 1 -> 0
Changed lines of the file:
@@
 	1    0    0    -1
 $EndComp
-NoConn ~ 6350 1600
 Wire Wire Line
 	6200 1200 6150 1200
@@
 P 9050 3550
 F 0 "R14" V 8843 3550 50  0000 C CNN
-F 1 "1k" V 8934 3550 50  0000 C CNN
+F 1 "1M" V 8934 3550 50  0000 C CNN
 F 2 "Resistor_SMD:R_0805_2012Metric" V 8980 3550 50  0001 C CNN
 F 3 "~" H 9050 3550 50  0001 C CNN
@@
 P 9050 4300
 F 0 "R15" V 8843 4300 50  0000 C CNN
-F 1 "1k" V 8934 4300 50  0000 C CNN
+F 1 "1M" V 8934 4300 50  0000 C CNN
 F 2 "Resistor_SMD:R_0805_2012Metric" V 8980 4300 50  0001 C CNN
 F 3 "~" H 9050 4300 50  0001 C CNN
@@
 P 4850 3350
 F 0 "J4" H 4930 3342 50  0000 L CNN
-F 1 "Conn_01x02" H 4930 3251 50  0000 L CNN
+F 1 "Conn_01x02" H 4930 3251 50  0001 L CNN
 F 2 "Connector_PinHeader_2.54mm:PinHeader_1x02_P2.54mm_Vertical" H 4850 3350 50  0001 C CNN
 F 3 "~" H 4850 3350 50  0001 C CNN
@@
 P 10150 1800
 F 0 "U3" H 10150 2167 50  0000 C CNN
-F 1 "Opamp_Quad_Generic" H 10150 2076 50  0000 C CNN
+F 1 "Opamp_Quad_Generic" H 10150 2076 50  0001 C CNN
 F 2 "Package_DIP:DIP-14_W7.62mm_Socket" H 10150 1800 50  0001 C CNN
 F 3 "~" H 10150 1800 50  0001 C CNN
@@
 P 2950 4550
 F 0 "U3" H 2950 4917 50  0000 C CNN
-F 1 "Opamp_Quad_Generic" H 2950 4826 50  0000 C CNN
+F 1 "Opamp_Quad_Generic" H 2950 4826 50  0001 C CNN
 F 2 "Package_DIP:DIP-14_W7.62mm_Socket" H 2950 4550 50  0001 C CNN
 F 3 "~" H 2950 4550 50  0001 C CNN
@@
 P 2950 4550
 F 0 "U3" H 2908 4596 50  0000 L CNN
-F 1 "Opamp_Quad_Generic" H 2908 4505 50  0000 L CNN
+F 1 "Opamp_Quad_Generic" H 2908 4505 50  0001 L CNN
 F 2 "Package_DIP:DIP-14_W7.62mm_Socket" H 2950 4550 50  0001 C CNN
 F 3 "~" H 2950 4550 50  0001 C CNN
@@
 U 4 1 5C02AE3C
 P 5550 3750
-F 0 "U5" H 5550 4117 50  0000 C CNN
-F 1 "Opamp_Quad_Generic" H 5550 4026 50  0000 C CNN
+F 0 "U5" H 5650 3900 50  0000 C CNN
+F 1 "Opamp_Quad_Generic" H 5550 4026 50  0001 C CNN
 F 2 "Package_DIP:DIP-14_W7.62mm_Socket" H 5550 3750 50  0001 C CNN
 F 3 "~" H 5550 3750 50  0001 C CNN
@@
 U 3 1 5C02AFF8
 P 6650 4400
-F 0 "U5" H 6650 4033 50  0000 C CNN
-F 1 "Opamp_Quad_Generic" H 6650 4124 50  0000 C CNN
+F 0 "U5" H 6650 4200 50  0000 C CNN
+F 1 "Opamp_Quad_Generic" H 6650 4124 50  0001 C CNN
 F 2 "Package_DIP:DIP-14_W7.62mm_Socket" H 6650 4400 50  0001 C CNN
 F 3 "~" H 6650 4400 50  0001 C CNN
@@
 P 9750 4400
 F 0 "U5" H 9708 4446 50  0000 L CNN
-F 1 "Opamp_Quad_Generic" H 9708 4355 50  0000 L CNN
+F 1 "Opamp_Quad_Generic" H 9708 4355 50  0001 L CNN
 F 2 "Package_DIP:DIP-14_W7.62mm_Socket" H 9750 4400 50  0001 C CNN
 F 3 "~" H 9750 4400 50  0001 C CNN

Commit message: Documentation added.
Connections:
- net labels removed: GNDA-power
Changed lines of the file:
@@
 P 10600 2350
 F 0 "J6" H 10680 2342 50  0000 L CNN
-F 1 "Conn_01x02" H 10680 2251 50  0000 L CNN
+F 1 "Conn_01x02" H 10680 2251 50  0001 L CNN
 F 2 "Connector_PinHeader_2.54mm:PinHeader_1x02_P2.54mm_Vertical" H 10600 2350 50  0001 C CNN
 F 3 "~" H 10600 2350 50  0001 C CNN
@@
 	1    10350 2700
 	1    0    0    1
-$EndComp
-$Comp
-L placa_aquisicao_e_filtros-rescue:GNDA-power #PWR026
-U 1 1 5C062DA4
-P 10350 2950
-F 0 "#PWR026" H 10350 2700 50  0001 C CNN
-F 1 "GNDA-power" H 10355 2777 50  0000 C CNN
-F 2 "" H 10350 2950 50  0001 C CNN
-F 3 "" H 10350 2950 50  0001 C CNN
-	1    10350 2950
-	-1   0    0    -1
 $EndComp
 Wire Wire Line
@@
 P 9750 4400
 F 0 "U5" H 9750 4767 50  0000 C CNN
-F 1 "Opamp_Quad_Generic" H 9750 4676 50  0000 C CNN
+F 1 "Opamp_Quad_Generic" H 9750 4676 50  0001 C CNN
 F 2 "Package_DIP:DIP-14_W7.62mm_Socket" H 9750 4400 50  0001 C CNN
 F 3 "~" H 9750 4400 50  0001 C CNN
@@
 U 1 1 5C02C8D3
 P 1950 2500
-F 0 "U2" H 2391 2546 50  0000 L CNN
-F 1 "TPS60401" H 2391 2455 50  0000 L CNN
+F 0 "U2" H 2350 2700 50  0000 L CNN
+F 1 "TPS60401" H 2350 2600 50  0000 L CNN
 F 2 "Package_TO_SOT_SMD:SOT-23-5" H 1950 2500 50  0001 C CNN
 F 3 "http://www.ti.com/lit/ds/symlink/tps60400.pdf" H 2600 1800 50  0001 C CNN
@@
 Wire Wire Line
 	10350 2900 10350 2950
+$Comp
+L power:GNDA #PWR?
+U 1 1 5C176ABF
+P 10350 2950
+F 0 "#PWR?" H 10350 2700 50  0001 C CNN
+F 1 "GNDA" H 10355 2777 50  0000 C CNN
+F 2 "" H 10350 2950 50  0001 C CNN
+F 3 "" H 10350 2950 50  0001 C CNN
+	1    10350 2950
+	1    0    0    -1
+$EndComp
 $EndSCHEMATC
