File: hardware/prototipo/placa_aquisicao_e_filtros/prototipo_inicial/placa_aquisicao_e_filtros.sch (KiCad schematic (older format))
At the start: 23 parts, among them J1 Conn_01x04, J3 Conn_01x02, J4 Conn_02x04_Counter_Clockwise, U1 Opamp_Quad_Generic, U2 AD620

Commit message: Documentation added.
Other:
- moved on the sheet: C1, C2, C3, C4, C5, J1, J3, J4, R1, R2, R3, R4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
